File: KiCad/CPU_block_diagram/_autosave-untitled.kicad_sch (KiCad schematic)
At the start: 6 parts, among them U1 LM555xN

Commit message: vault backup: 2025-12-28 23:13:10
Parts:
- removed C1: 0.01µF, symbol Device:C
- removed C2: 1µF, symbol Device:C_Polarized_US
- removed R1, R2: 1K, symbol Device:R_US
- removed RV1: 1M, symbol Device:R_Potentiometer_US
- removed U1: LM555xN, Package_DIP:DIP-8_W7.62mm, symbol Timer:LM555xN
- added C3: 1µF, symbol Device:C_Polarized_US
- added C4: 0.01µF, symbol Device:C
- added R3, R4: 1K, symbol Device:R_US
- added RV2: 1M, symbol Device:R_Potentiometer_US
- added U2: LM555xN, Package_DIP:DIP-8_W7.62mm, symbol Timer:LM555xN
Connections:
- net GND: now also C3.1, C3.2, C4.1, RV2.3, U2.1 (GND), U2.2 (TRIG), U2.6 (THRES)
- net VCC: now also R4.1, U2.4 (~{RST}), U2.8 (VCC)
- new net: C4.2, U2.5 (CONT)
- new net: R3.1, R4.2, U2.7 (DISCH)
- new net: R3.2, RV2.2
Other:
- removed sheet Astable Mode
