File: KiCad/CPU_block_diagram/clock_module.kicad_sch (KiCad schematic)
At the start: 6 parts, among them U1 LM555xN

Commit message: vault backup: 2025-12-29 00:49:08
Parts:
- removed C1: 0.01µF, symbol Device:C
- removed C2: 1µF, symbol Device:C_Polarized_US
- removed R1, R2: 1K, symbol Device:R_US
- removed RV1: 1M, symbol Device:R_Potentiometer_US
- removed U1: LM555xN, Package_DIP:DIP-8_W7.62mm, symbol Timer:LM555xN
- added C3: 1µF, symbol Device:C_Polarized_US
- added C4: 0.01µF, symbol Device:C
- added R3, R4: 1K, symbol Device:R_US
- added RV2: 1M, symbol Device:R_Potentiometer_US
- added U2: LM555xN, Package_DIP:DIP-8_W7.62mm, symbol Timer:LM555xN
Connections:
- net GND: now also C3.1, C3.2, C4.1, RV2.3, U2.1 (GND), U2.2 (TRIG), U2.6 (THRES)
- net VCC: now also R4.1, U2.4 (~{RST}), U2.8 (VCC)
- new net: R3.1, R4.2, U2.7 (DISCH)
- new net: C4.2, U2.5 (CONT)
- new net: R3.2, RV2.2
Other:
- removed sheet Astable Mode

Commit message: vault backup: 2025-12-29 04:12:58
Connections:
- net GND: no longer C3.1, RV2.3, U2.2 (TRIG), U2.6 (THRES)
- net at RV2.1: now also C3.1, U2.2 (TRIG), U2.6 (THRES)
Other:
- moved on the sheet: C3, R3, R4, RV2

Commit message: vault backup: 2025-12-29 04:43:05
Parts:
- added D1: LED, symbol Device:LED
- added R1: R_US, symbol Device:R_US
Connections:
- net GND: now also R1.2
- net at U2.3 (OUT): now also D1.2 (A)
- net VCC renamed +5V
- new net: D1.1 (K), R1.1
- no-connect marks 0 -> 1
Other:
- title: (none) -> 8-Bit Computer

Commit message: vault backup: 2025-12-29 05:43:18
Parts:
- removed D1: LED, symbol Device:LED
- added C2, C6, C7: 0.01µF, symbol Device:C
- added C5: 1µF, symbol Device:C_Polarized_US
- added R2: 1M, symbol Device:R_US
- added R5, R6: 1K, symbol Device:R_US
- added SW1: SW_Push, symbol Switch:SW_Push
- added U1, U3: LM555xN, Package_DIP:DIP-8_W7.62mm, symbol Timer:LM555xN
- R1: value R_US -> 1K
Connections:
- net +5V: now also R1.1, R2.1, R6.1, U1.4 (~{RST}), U1.8 (VCC), U3.4 (~{RST}), U3.8 (VCC)
- net GND: now also C2.1, C5.2, C6.1, C7.1, SW1.1, U1.1 (GND), U3.1 (GND); no longer R1.2
- net AstableMode: now reaches U2.3 (OUT)
- new net: R5.1, R6.2, U3.7 (DISCH)
- new net: C5.1, U3.2 (TRIG), U3.6 (THRES)
- new net: C6.2, U3.5 (CONT)
- new net: C7.2, R1.2, R2.2, SW1.2, U1.2 (TRIG), U1.6 (THRES), U1.7 (DISCH)
- new net: C2.2, U1.5 (CONT)
- new net BiStableMode: U1.3 (OUT)
Other:
- note added: "Astable Mode"
- note added: "Bi-Stable Mode (Debouncer)"
- title: 8-Bit Computer -> Clock Module
- moved on the sheet: C3, C4, R3, R4, RV2, U2

Commit message: vault backup: 2025-12-29 10:56:26
Parts:
- removed C5: 1µF, symbol Device:C_Polarized_US
- added SW2: SW_SPDT, symbol Switch:SW_SPDT
Connections:
- net +5V: now also R5.1; no longer U3.4 (~{RST})
- net GND: now also U3.6 (THRES), SW2.2 (B)
- net at U3.2 (TRIG): now also R5.2, SW2.1 (A); no longer U3.6 (THRES)
- net MonoStableMode: now reaches U3.3 (OUT)
- new net: R6.2, SW2.3 (C), U3.4 (~{RST})
- now unconnected: U3.7 (DISCH)
- no-connect marks 1 -> 2
Other:
- note added: "Mono-Stable Mode"
- moved on the sheet: C2, C7, R1, R2, R5, R6, SW1, U1

Commit message: vault backup: 2025-12-29 13:43:32
Parts:
- removed SW1: SW_Push, symbol Switch:SW_Push
- removed SW2: SW_SPDT, symbol Switch:SW_SPDT
Connections:
- net RESET_N: now reaches R6.2, U3.4 (~{RST})
- net TRIGGER_N: now reaches R5.2, U3.2 (TRIG)
- net STEP_CLK: now reaches C7.2, R1.2, R2.2, U1.2 (TRIG), U1.6 (THRES), U1.7 (DISCH)

Commit message: vault backup: 2025-12-29 14:13:42
Parts:
- added U1: 74LS04, symbol 74xx:74LS04
- added U2: 74LS08, symbol 74xx:74LS08
- added U3: 74LS32, symbol 74xx:74LS32
- renumbered C3 to C1, C4 to C2, C7 to C3, C2 to C4, C6 to C5, R3 to R1, R4 to R2, R1 to R3, R2 to R4, RV2 to RV1, U2 to U4, U1 to U5, U3 to U6
Connections:
- net +5V: now also U1.14 (VCC), U2.14 (VCC), U3.14 (VCC)
- net AstableMode: now also U2.4
- net BiStableMode: now also U2.2
- net GND: now also U1.7 (GND), U2.7 (GND), U3.7 (GND)
- net MonoStableMode: now also U1.1, U2.5
- new net: U1.2, U2.1
- new net: U2.6, U3.1
- new net: U2.3, U3.2
- new net: U2.9, U3.3
- new net: U1.4, U2.10
- new net CLK: U1.5, U2.8
- new net HLT: U1.3
- new net ~{CLK}: U1.6
Other:
- note added: "Logic"
- note added: "Logic Power"

Commit message: vault backup: 2025-12-30 00:26:07
Parts:
- renumbered U4 to U2, U2 to U3, U3 to U4
Changed lines of the file:
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@@
 		(on_board yes)
 		(dnp no)
-		(property "Reference" "U4"
+		(property "Reference" "U2"
 			(at 89.154 43.688 0)
 			(effects
@@
 			(project "CPU_block_diagram"
 				(path "/5324683e-15fd-4fa9-8f28-7726564ef1dc/23156860-93e6-4eb1-8f6c-79601c8beb45"
-					(reference "U4")
+					(reference "U2")
 					(unit 1)
 				)
@@
 		(dnp no)
 		(fields_autoplaced yes)
-		(property "Reference" "U2"
+		(property "Reference" "U3"
 			(at 88.8917 90.17 0)
 			(effects
@@
 			(project ""
 				(path "/5324683e-15fd-4fa9-8f28-7726564ef1dc/23156860-93e6-4eb1-8f6c-79601c8beb45"
-					(reference "U2")
+					(reference "U3")
 					(unit 2)
 				)
@@
 		(dnp no)
 		(fields_autoplaced yes)
-		(property "Reference" "U2"
+		(property "Reference" "U3"
 			(at 218.44 110.4899 0)
 			(effects
@@
 			(project ""
 				(path "/5324683e-15fd-4fa9-8f28-7726564ef1dc/23156860-93e6-4eb1-8f6c-79601c8beb45"
-					(reference "U2")
+					(reference "U3")
 					(unit 5)
 				)
@@
 		(dnp no)
 		(fields_autoplaced yes)
-		(property "Reference" "U3"
+		(property "Reference" "U4"
 			(at 238.76 110.4899 0)
 			(effects
@@
 			(project ""
 				(path "/5324683e-15fd-4fa9-8f28-7726564ef1dc/23156860-93e6-4eb1-8f6c-79601c8beb45"
-					(reference "U3")
+					(reference "U4")
 					(unit 5)
 				)
@@
 		(dnp no)
 		(fields_autoplaced yes)
-		(property "Reference" "U3"
+		(property "Reference" "U4"
 			(at 110.49 97.79 0)
 			(effects
@@
 			(project ""
 				(path "/5324683e-15fd-4fa9-8f28-7726564ef1dc/23156860-93e6-4eb1-8f6c-79601c8beb45"
-					(reference "U3")
+					(reference "U4")
 					(unit 1)
 				)
@@
 		(dnp no)
 		(fields_autoplaced yes)
-		(property "Reference" "#PWR06"
+		(property "Reference" "#PWR011"
 			(at 241.3 36.83 0)
 			(effects
@@
 			(project "CPU_block_diagram"
 				(path "/5324683e-15fd-4fa9-8f28-7726564ef1dc/23156860-93e6-4eb1-8f6c-79601c8beb45"
-					(reference "#PWR06")
+					(reference "#PWR011")
 					(unit 1)
 				)
@@
 		(dnp no)
 		(fields_autoplaced yes)
-		(property "Reference" "#PWR05"
+		(property "Reference" "#PWR010"
 			(at 238.76 77.47 0)
 			(effects
@@
 			(project "CPU_block_diagram"
 				(path "/5324683e-15fd-4fa9-8f28-7726564ef1dc/23156860-93e6-4eb1-8f6c-79601c8beb45"
-					(reference "#PWR05")
+					(reference "#PWR010")
 					(unit 1)
 				)
@@
 		(dnp no)
 		(fields_autoplaced yes)
-		(property "Reference" "U2"
+		(property "Reference" "U3"
 			(at 137.1517 100.33 0)
 			(effects
@@
 			(project ""
 				(path "/5324683e-15fd-4fa9-8f28-7726564ef1dc/23156860-93e6-4eb1-8f6c-79601c8beb45"
-					(reference "U2")
+					(reference "U3")
 					(unit 3)
 				)
@@
 		(dnp no)
 		(fields_autoplaced yes)
-		(property "Reference" "#PWR03"
+		(property "Reference" "#PWR06"
 			(at 157.48 77.47 0)
 			(effects
@@
 			(project "CPU_block_diagram"
 				(path "/5324683e-15fd-4fa9-8f28-7726564ef1dc/23156860-93e6-4eb1-8f6c-79601c8beb45"
-					(reference "#PWR03")
+					(reference "#PWR06")
 					(unit 1)
 				)
@@
 		(dnp no)
 		(fields_autoplaced yes)
-		(property "Reference" "#PWR01"
+		(property "Reference" "#PWR04"
 			(at 76.2 77.47 0)
 			(effects
@@
 			(project "CPU_block_diagram"
 				(path "/5324683e-15fd-4fa9-8f28-7726564ef1dc/23156860-93e6-4eb1-8f6c-79601c8beb45"
-					(reference "#PWR01")
+					(reference "#PWR04")
 					(unit 1)
 				)
@@
 		(dnp no)
 		(fields_autoplaced yes)
-		(property "Reference" "U2"
+		(property "Reference" "U3"
 			(at 88.8917 106.68 0)
 			(effects
@@
 			(project ""
 				(path "/5324683e-15fd-4fa9-8f28-7726564ef1dc/23156860-93e6-4eb1-8f6c-79601c8beb45"
-					(reference "U2")
+					(reference "U3")
 					(unit 1)
 				)
@@
 		(dnp no)
 		(fields_autoplaced yes)
-		(property "Reference" "#PWR04"
+		(property "Reference" "#PWR07"
 			(at 160.02 36.83 0)
 			(effects
@@
 			(project "CPU_block_diagram"
 				(path "/5324683e-15fd-4fa9-8f28-7726564ef1dc/23156860-93e6-4eb1-8f6c-79601c8beb45"
-					(reference "#PWR04")
+					(reference "#PWR07")
 					(unit 1)
 				)
@@
 		(dnp no)
 		(fields_autoplaced yes)
-		(property "Reference" "#PWR09"
+		(property "Reference" "#PWR08"
 			(at 212.09 100.33 0)
 			(effects
@@
 			(project ""
 				(path "/5324683e-15fd-4fa9-8f28-7726564ef1dc/23156860-93e6-4eb1-8f6c-79601c8beb45"
-					(reference "#PWR09")
+					(reference "#PWR08")
 					(unit 1)
 				)
@@
 		(dnp no)
 		(fields_autoplaced yes)
-		(property "Reference" "#PWR010"
+		(property "Reference" "#PWR09"
 			(at 212.09 133.35 0)
 			(effects
@@
 			(project ""
 				(path "/5324683e-15fd-4fa9-8f28-7726564ef1dc/23156860-93e6-4eb1-8f6c-79601c8beb45"
-					(reference "#PWR010")
+					(reference "#PWR09")
 					(unit 1)
 				)
@@
 		(dnp no)
 		(fields_autoplaced yes)
-		(property "Reference" "#PWR02"
+		(property "Reference" "#PWR05"
 			(at 78.74 36.83 0)
 			(effects
@@
 			(project ""
 				(path "/5324683e-15fd-4fa9-8f28-7726564ef1dc/23156860-93e6-4eb1-8f6c-79601c8beb45"
-					(reference "#PWR02")
-					(unit 1)
-				)
+					(reference "#PWR05")
+					(unit 1)
+				)
