File: KiCad/CPU_block_diagram/_autosave-a_register.kicad_sch (KiCad schematic)
At the start: 19 parts, among them U7 74LS245, U8 74LS173, U9 74LS173

Commit message: vault backup: 2026-01-02 19:39:35
Connections:
- net BUS0: now reaches U9.11 (D3)
- net BUS0: now also U7.11 (B7)
- net BUS1: now reaches U9.12 (D2)
- net BUS1: now also U7.12 (B6)
- net BUS2: now reaches U9.13 (D1)
- net BUS2: now also U7.13 (B5)
- net BUS3: now reaches U9.14 (D0)
- net BUS3: now also U7.14 (B4)
- net BUS4: now reaches U8.11 (D3)
- net BUS4: now also U7.15 (B3)
- net BUS5: now reaches U8.12 (D2)
- net BUS5: now also U7.16 (B2)
- net BUS6: now reaches U8.13 (D1)
- net BUS6: now also U7.17 (B1)
- net BUS7: now reaches U8.14 (D0)
- net BUS7: now also U7.18 (B0)
Other:
- moved on the sheet: U7, U8, U9
