File: KiCad/CPU_block_diagram/CPU_block_diagram.kicad_sch (KiCad schematic)
At the start: 0 parts

Commit message: vault backup: 2025-12-29 00:49:08
Parts:
- added C1: 0.01µF, symbol Device:C
- added C2: 1µF, symbol Device:C_Polarized_US
- added R1, R2: 1K, symbol Device:R_US
- added RV1: 1M, symbol Device:R_Potentiometer_US
- added U1: LM555xN, Package_DIP:DIP-8_W7.62mm, symbol Timer:LM555xN
Connections:
- new net: C1.2, U1.5 (CONT)
- new net: R1.2, R2.1, U1.7 (DISCH)
- new net: R2.2, RV1.2
- new net GND: C1.1, C2.1, C2.2, RV1.3, U1.1 (GND), U1.2 (TRIG), U1.6 (THRES)
- new net VCC: R1.1, U1.4 (~{RST}), U1.8 (VCC)
Other:
- added sheet Clock Module (clock_module.kicad_sch)
- note added: "8 Bit Computer"

Commit message: vault backup: 2025-12-29 04:12:58
Parts:
- removed C1: 0.01µF, symbol Device:C
- removed C2: 1µF, symbol Device:C_Polarized_US
- removed R1, R2: 1K, symbol Device:R_US
- removed RV1: 1M, symbol Device:R_Potentiometer_US
- removed U1: LM555xN, Package_DIP:DIP-8_W7.62mm, symbol Timer:LM555xN
Other:
- note added: "8 Bit Computer Top Level"
- note removed: "8 Bit Computer"

Commit message: vault backup: 2025-12-29 05:43:18
Other:
- added sheet Power (power.kicad_sch)
Changed lines of the file:
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@@
 	)
 	(sheet
-		(at 21.59 25.4)
+		(at 20.32 48.26)
 		(size 35.56 22.86)
 		(exclude_from_sim no)
@@
 		)
 		(property "Sheetname" "Clock Module"
-			(at 21.59 24.6884 0)
+			(at 20.32 47.5484 0)
 			(effects
 				(font
@@
 		)
 		(property "Sheetfile" "clock_module.kicad_sch"
-			(at 21.59 48.8446 0)
+			(at 20.32 71.7046 0)
 			(effects
 				(font
@@
 				)
 			)
+		)
+	)
+	(sheet
+		(at 20.32 25.4)
+		(size 36.83 15.24)
+		(exclude_from_sim no)
+		(in_bom yes)
+		(on_board yes)
+		(dnp no)
+		(fields_autoplaced yes)
+		(stroke
+			(width 0.1524)
+			(type solid)
+		)
+		(fill
+			(color 0 0 0 0.0000)
+		)
+		(property "Sheetname" "Power"
+			(at 20.32 24.6884 0)
+			(effects
+				(font
+					(size 1.27 1.27)
+				)
+				(justify left bottom)
+			)
+		)
+		(property "Sheetfile" "power.kicad_sch"
+			(at 20.32 41.2246 0)
+			(effects
+				(font
+					(size 1.27 1.27)
+				)
+				(justify left top)
+			)
+		)
+		(instances
+			(project "CPU_block_diagram"
+				(path "/5324683e-15fd-4fa9-8f28-7726564ef1dc"
+					(page "3")
+				)
+			)

Commit message: vault backup: 2025-12-29 14:13:42
Parts:
- added SW1: SW_Push, symbol Switch:SW_Push
- added SW2: SW_SPDT, symbol Switch:SW_SPDT
Connections:
- new net Clock Module/RESET_N: SW2.1 (A)
- new net Clock Module/STEP_CLK: SW1.2
- new net Clock Module/TRIGGER_N: SW2.3 (C)
- new net GND: SW1.1, SW2.2 (B)
Other:
- sheet Clock Module ports: added CLK, HLT, RESET_N, STEP_CLK, TRIGGER_N, ~{CLK}; removed none

Commit message: vault backup: 2025-12-30 00:26:07
Other:
- moved on the sheet: SW1, SW2
Changed lines of the file:
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@@
 	)
 	(junction
-		(at 76.2 78.74)
+		(at 76.2 81.28)
 		(diameter 0)
 		(color 0 0 0 0)
@@
 	(wire
 		(pts
-			(xy 64.77 67.31) (xy 57.15 67.31)
-		)
-		(stroke
-			(width 0)
-			(type default)
-		)
-	)
-	(wire
-		(pts
-			(xy 76.2 78.74) (xy 73.66 78.74)
-		)
-		(stroke
-			(width 0)
-			(type default)
-		)
-	)
-	(wire
-		(pts
-			(xy 63.5 78.74) (xy 59.69 78.74)
-		)
-		(stroke
-			(width 0)
-			(type default)
-		)
-	)
-	(wire
-		(pts
-			(xy 59.69 71.12) (xy 59.69 78.74)
+			(xy 64.77 74.93) (xy 62.23 74.93)
+		)
+		(stroke
+			(width 0)
+			(type default)
+		)
+	)
+	(wire
+		(pts
+			(xy 63.5 62.23) (xy 57.15 62.23)
+		)
+		(stroke
+			(width 0)
+			(type default)
+		)
+	)
+	(wire
+		(pts
+			(xy 76.2 81.28) (xy 73.66 81.28)
+		)
+		(stroke
+			(width 0)
+			(type default)
+		)
+	)
+	(wire
+		(pts
+			(xy 63.5 81.28) (xy 59.69 81.28)
+		)
+		(stroke
+			(width 0)
+			(type default)
+		)
+	)
+	(wire
+		(pts
+			(xy 62.23 67.31) (xy 57.15 67.31)
+		)
+		(stroke
+			(width 0)
+			(type default)
+		)
+	)
+	(wire
+		(pts
+			(xy 59.69 71.12) (xy 59.69 81.28)
+		)
+		(stroke
+			(width 0)
+			(type default)
+		)
+	)
+	(wire
+		(pts
+			(xy 62.23 74.93) (xy 62.23 67.31)
 		)
 		(stroke
@@
 	(wire
 		(pts
-			(xy 76.2 64.77) (xy 76.2 78.74)
-		)
-		(stroke
-			(width 0)
-			(type default)
-		)
-	)
-	(wire
-		(pts
-			(xy 64.77 62.23) (xy 57.15 62.23)
-		)
-		(stroke
-			(width 0)
-			(type default)
-		)
-	)
-	(wire
-		(pts
-			(xy 74.93 64.77) (xy 76.2 64.77)
-		)
-		(stroke
-			(width 0)
-			(type default)
-		)
-	)
-	(wire
-		(pts
-			(xy 76.2 78.74) (xy 76.2 82.55)
+			(xy 76.2 72.39) (xy 76.2 81.28)
+		)
+		(stroke
+			(width 0)
+			(type default)
+		)
+	)
+	(wire
+		(pts
+			(xy 64.77 69.85) (xy 63.5 69.85)
+		)
+		(stroke
+			(width 0)
+			(type default)
+		)
+	)
+	(wire
+		(pts
+			(xy 74.93 72.39) (xy 76.2 72.39)
+		)
+		(stroke
+			(width 0)
+			(type default)
+		)
+	)
+	(wire
+		(pts
+			(xy 57.15 58.42) (xy 72.39 58.42)
+		)
+		(stroke
+			(width 0)
+			(type default)
+		)
+	)
+	(wire
+		(pts
+			(xy 76.2 81.28) (xy 76.2 82.55)
+		)
+		(stroke
+			(width 0)
+			(type default)
+		)
+	)
+	(wire
+		(pts
+			(xy 63.5 69.85) (xy 63.5 62.23)
 		)
 		(stroke
@@
 	(symbol
 		(lib_id "Switch:SW_SPDT")
-		(at 69.85 64.77 0)
+		(at 69.85 72.39 0)
 		(mirror y)
 		(unit 1)
@@
 		(fields_autoplaced yes)
 		(property "Reference" "SW2"
-			(at 69.85 55.88 0)
+			(at 69.85 63.5 0)
 			(effects
 				(font
@@
 		)
 		(property "Value" "SW_SPDT"
-			(at 69.85 58.42 0)
+			(at 69.85 66.04 0)
 			(effects
 				(font
@@
 		)
 		(property "Footprint" ""
-			(at 69.85 64.77 0)
+			(at 69.85 72.39 0)
 			(effects
 				(font
@@
 		)
 		(property "Datasheet" "~"
+			(at 69.85 80.01 0)
+			(effects
+				(font
+					(size 1.27 1.27)
+				)
+				(hide yes)
+			)
+		)
+		(property "Description" "Switch, single pole double throw"
 			(at 69.85 72.39 0)
-			(effects
-				(font
-					(size 1.27 1.27)
-				)
-				(hide yes)
-			)
-		)
-		(property "Description" "Switch, single pole double throw"
-			(at 69.85 64.77 0)
 			(effects
 				(font
@@
 	(symbol
 		(lib_id "Switch:SW_Push")
-		(at 68.58 78.74 0)
+		(at 68.58 81.28 0)
 		(mirror y)
 		(unit 1)
@@
 		(on_board yes)
 		(dnp no)
-		(fields_autoplaced yes)
 		(property "Reference" "SW1"
-			(at 68.58 71.12 0)
+			(at 68.58 83.312 0)
 			(effects
 				(font
@@
 		)
 		(property "Value" "SW_Push"
-			(at 68.58 73.66 0)
+			(at 68.58 85.852 0)
 			(effects
 				(font
@@
 		)
 		(property "Footprint" ""
-			(at 68.58 73.66 0)
+			(at 68.58 76.2 0)
 			(effects
 				(font
@@
 		)
 		(property "Datasheet" "~"
-			(at 68.58 73.66 0)
+			(at 68.58 76.2 0)
 			(effects
 				(font
@@
 		)
 		(property "Description" "Push button switch, generic, two pins"
-			(at 68.58 78.74 0)
+			(at 68.58 81.28 0)
 			(effects
 				(font
@@
 				(path "/5324683e-15fd-4fa9-8f28-7726564ef1dc"
 					(reference "SW1")
+					(unit 1)
+				)
+			)
+		)
+	)
+	(symbol
+		(lib_id "power:+5V")
+		(at 72.39 58.42 0)
+		(unit 1)
+		(exclude_from_sim no)
+		(in_bom yes)
+		(on_board yes)
+		(dnp no)
+		(fields_autoplaced yes)
+		(property "Reference" "#PWR012"
+			(at 72.39 62.23 0)
+			(effects
+				(font
+					(size 1.27 1.27)
+				)
+				(hide yes)
+			)
+		)
+		(property "Value" "+5V"
+			(at 72.39 53.34 0)
+			(effects
+				(font
+					(size 1.27 1.27)
+				)
+			)
+		)
+		(property "Footprint" ""
+			(at 72.39 58.42 0)
+			(effects
+				(font
+					(size 1.27 1.27)
+				)
+				(hide yes)
+			)
+		)
+		(property "Datasheet" ""
+			(at 72.39 58.42 0)
+			(effects
+				(font
+					(size 1.27 1.27)
+				)
+				(hide yes)
+			)
+		)
+		(property "Description" "Power symbol creates a global label with name \"+5V\""
+			(at 72.39 58.42 0)
+			(effects
+				(font
+					(size 1.27 1.27)
+				)
+				(hide yes)
+			)
+		)
+		(pin "1"
+		)
+		(instances
+			(project ""
+				(path "/5324683e-15fd-4fa9-8f28-7726564ef1dc"
+					(reference "#PWR012")
 					(unit 1)
 				)
@@
 		(dnp no)
 		(fields_autoplaced yes)
-		(property "Reference" "#PWR011"
+		(property "Reference" "#PWR01"
 			(at 76.2 88.9 0)
 			(effects
@@
 			(project ""
 				(path "/5324683e-15fd-4fa9-8f28-7726564ef1dc"
-					(reference "#PWR011")
+					(reference "#PWR01")
 					(unit 1)
 				)

Commit message: vault backup: 2025-12-30 22:01:07
Parts:
- added D1: RED_LED, symbol Device:LED
- added R1: 220, symbol Device:R_US
- added RV1: 1M, symbol Device:R_Potentiometer_US
- renumbered SW2 to SW1, SW1 to SW2
Connections:
- net Clock Module/CLK: now also R1.2
- net GND: now also D1.1 (K)
- new net: D1.2 (A), R1.1
- new net Clock Module/FREQ_ADJ_A: RV1.2
- new net Clock Module/FREQ_ADJ_B: RV1.3
- no-connect marks 0 -> 1
Other:
- sheet Clock Module ports: added FREQ_ADJ_A, FREQ_ADJ_B; removed none
- moved on the sheet: SW1, SW2

Commit message: vault backup: 2026-01-03 00:49:48
Other:
- added sheet A Register (a_register.kicad_sch)
- added sheet B Register (b_register.kicad_sch)
Changed lines of the file:
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@@
+	)
+	(sheet
+		(at 73.66 99.06)
+		(size 35.56 30.48)
+		(exclude_from_sim no)
+		(in_bom yes)
+		(on_board yes)
+		(dnp no)
+		(fields_autoplaced yes)
+		(stroke
+			(width 0.1524)
+			(type solid)
+		)
+		(fill
+			(color 0 0 0 0.0000)
+		)
+		(property "Sheetname" "B Register"
+			(at 73.66 98.3484 0)
+			(effects
+				(font
+					(size 1.27 1.27)
+				)
+				(justify left bottom)
+			)
+		)
+		(property "Sheetfile" "b_register.kicad_sch"
+			(at 73.66 130.1246 0)
+			(effects
+				(font
+					(size 1.27 1.27)
+				)
+				(justify left top)
+			)
+		)
+		(instances
+			(project "CPU_block_diagram"
+				(path "/5324683e-15fd-4fa9-8f28-7726564ef1dc"
+					(page "5")
+				)
+			)
+		)
 	)
 	(sheet
@@
 				)
 			)
+		)
+	)
+	(sheet
+		(at 30.48 97.79)
+		(size 33.02 30.48)
+		(exclude_from_sim no)
+		(in_bom yes)
+		(on_board yes)
+		(dnp no)
+		(fields_autoplaced yes)
+		(stroke
+			(width 0.1524)
+			(type solid)
+		)
+		(fill
+			(color 0 0 0 0.0000)
+		)
+		(property "Sheetname" "A Register"
+			(at 30.48 97.0784 0)
+			(effects
+				(font
+					(size 1.27 1.27)
+				)
+				(justify left bottom)
+			)
+		)
+		(property "Sheetfile" "a_register.kicad_sch"
+			(at 30.48 128.8546 0)
+			(effects
+				(font
+					(size 1.27 1.27)
+				)
+				(justify left top)
+			)
+		)
+		(instances
+			(project "CPU_block_diagram"
+				(path "/5324683e-15fd-4fa9-8f28-7726564ef1dc"
+					(page "4")
+				)
+			)

Commit message: vault backup: 2026-01-03 05:38:52
Changed lines of the file:
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@@
-	)
-	(sheet
-		(at 73.66 99.06)
-		(size 35.56 30.48)
-		(exclude_from_sim no)
-		(in_bom yes)
-		(on_board yes)
-		(dnp no)
-		(fields_autoplaced yes)
-		(stroke
-			(width 0.1524)
-			(type solid)
-		)
-		(fill
-			(color 0 0 0 0.0000)
-		)
-		(property "Sheetname" "B Register"
-			(at 73.66 98.3484 0)
-			(effects
-				(font
-					(size 1.27 1.27)
-				)
-				(justify left bottom)
-			)
-		)
-		(property "Sheetfile" "b_register.kicad_sch"
-			(at 73.66 130.1246 0)
-			(effects
-				(font
-					(size 1.27 1.27)
-				)
-				(justify left top)
-			)
-		)
-		(instances
-			(project "CPU_block_diagram"
-				(path "/5324683e-15fd-4fa9-8f28-7726564ef1dc"
-					(page "5")
-				)
-			)
-		)
 	)
 	(sheet
@@
 				)
 			)
+		)
+	)
+	(sheet
+		(at 78.74 97.79)
+		(size 33.02 30.48)
+		(exclude_from_sim no)
+		(in_bom yes)
+		(on_board yes)
+		(dnp no)
+		(fields_autoplaced yes)
+		(stroke
+			(width 0.1524)
+			(type solid)
+		)
+		(fill
+			(color 0 0 0 0.0000)
+		)
+		(property "Sheetname" "B Register"
+			(at 78.74 97.0784 0)
+			(effects
+				(font
+					(size 1.27 1.27)
+				)
+				(justify left bottom)
+			)
+		)
+		(property "Sheetfile" "b_register.kicad_sch"
+			(at 78.74 128.8546 0)
+			(effects
+				(font
+					(size 1.27 1.27)
+				)
+				(justify left top)
+			)
+		)
+		(instances
+			(project "CPU_block_diagram"
+				(path "/5324683e-15fd-4fa9-8f28-7726564ef1dc"
+					(page "6")
+				)
+			)
