File: KiCad/CPU_block_diagram/CPU_block_diagram.kicad_sch (KiCad schematic)
At the start: 5 parts, among them SW1 SW_SPDT, SW2 SW_Push

Commit message: vault backup: 2026-01-03 13:53:37
Other:
- added sheet Instruction Register (IR_register.kicad_sch)
Changed lines of the file:
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@@
 	)
 	(sheet
-		(at 78.74 97.79)
-		(size 33.02 30.48)
+		(at 72.39 97.79)
+		(size 29.21 30.48)
 		(exclude_from_sim no)
 		(in_bom yes)
@@
 		)
 		(property "Sheetname" "B Register"
-			(at 78.74 97.0784 0)
+			(at 72.39 97.0784 0)
 			(effects
 				(font
@@
 		)
 		(property "Sheetfile" "b_register.kicad_sch"
-			(at 78.74 128.8546 0)
+			(at 72.39 128.8546 0)
 			(effects
 				(font
+					(size 1.27 1.27)
+				)
+				(justify left top)
+			)
+		)
+		(instances
+			(project "CPU_block_diagram"
+				(path "/5324683e-15fd-4fa9-8f28-7726564ef1dc"
+					(page "5")
+				)
+			)
+		)
+	)
+	(sheet
+		(at 107.95 97.79)
+		(size 31.75 30.48)
+		(exclude_from_sim no)
+		(in_bom yes)
+		(on_board yes)
+		(dnp no)
+		(fields_autoplaced yes)
+		(stroke
+			(width 0.1524)
+			(type solid)
+		)
+		(fill
+			(color 0 0 0 0.0000)
+		)
+		(property "Sheetname" "Instruction Register"
+			(at 107.95 97.0784 0)
+			(effects
+				(font
+					(size 1.27 1.27)
+				)
+				(justify left bottom)
+			)
+		)
+		(property "Sheetfile" "IR_register.kicad_sch"
+			(at 107.95 128.8546 0)
+			(effects
+				(font

Commit message: vault backup: 2026-01-03 15:04:01
Parts:
- removed D1: RED_LED, symbol Device:LED
- removed R1: 220, symbol Device:R_US
- removed RV1: 1M, symbol Device:R_Potentiometer_US
- removed SW1: SW_SPDT, symbol Switch:SW_SPDT
- removed SW2: SW_Push, symbol Switch:SW_Push
Connections:
- no-connect marks 1 -> 0
Other:
- sheet A Register ports: added A0, A1, A2, A3, A4, A5, A6, A7, BUS0, BUS1, BUS2, BUS3, BUS4, BUS5, BUS6, BUS7, CLK, CLR, ~{AI}, ~{AO}; removed none
- sheet B Register ports: added B0, B1, B2, B3, B4, B5, B6, B7, BUS0, BUS1, BUS2, BUS3, BUS4, BUS5, BUS6, BUS7, CLK, CLR, ~{BI}, ~{BO}; removed none
- sheet Clock Module ports: added none; removed FREQ_ADJ_A, FREQ_ADJ_B, RESET_N, STEP_CLK, TRIGGER_N
- sheet Instruction Register ports: added BUS0, BUS1, BUS2, BUS3, BUS4, BUS5, BUS6, BUS7, CLK, CLR, IR4, IR5, IR6, IR7, ~{IRI}, ~{IRO}; removed none

Commit message: vault backup: 2026-01-03 15:51:55
Other:
- sheet Instruction Register: file IR_register.kicad_sch -> ir_register.kicad_sch
- note added: "CLOCK"
- note added: "POWER"
- note added: "REGISTERS"
- note removed: "8 Bit Computer Top Level"

Commit message: vault backup: 2026-01-05 18:47:29
Parts:
- added D26, D27, D28, D29, D30, D31, D32, D33: RED, symbol Device:LED
- added R32, R33, R34, R35, R36, R37, R38, R39: 220, symbol Device:R_US
- added R40, R41, R42, R43, R44, R45, R46, R47: 10K, symbol Device:R_US
Connections:
- net A Register/BUS0: now also D33.2 (A), R47.1
- net A Register/BUS1: now also D32.2 (A), R46.1
- net A Register/BUS2: now also D31.2 (A), R45.1
- net A Register/BUS3: now also D30.2 (A), R44.1
- net A Register/BUS4: now also D29.2 (A), R43.1
- net A Register/BUS5: now also D28.2 (A), R42.1
- net A Register/BUS6: now also D27.2 (A), R41.1
- net A Register/BUS7: now also D26.2 (A), R40.1
- new net: D33.1 (K), R39.1
- new net: D26.1 (K), R32.1
- new net: D31.1 (K), R37.1
- new net: D29.1 (K), R35.1
- new net: D28.1 (K), R34.1
- new net: D32.1 (K), R38.1
- new net: D30.1 (K), R36.1
- new net: D27.1 (K), R33.1
- new net GND: R32.2, R33.2, R34.2, R35.2, R36.2, R37.2, R38.2, R39.2, R40.2, R41.2, R42.2, R43.2, R44.2, R45.2, R46.2, R47.2
Other:
- note added: "BUS"
- note added: "OUTPUT"

Commit message: vault backup: 2026-01-10 22:03:55
Other:
- added sheet Arithmetic Logic Unit (alu.kicad_sch)
Changed lines of the file:
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@@
+	)
+	(sheet
+		(at 85.09 50.8)
+		(size 29.21 30.48)
+		(exclude_from_sim no)
+		(in_bom yes)
+		(on_board yes)
+		(dnp no)
+		(fields_autoplaced yes)
+		(stroke
+			(width 0.1524)
+			(type solid)
+		)
+		(fill
+			(color 0 0 0 0.0000)
+		)
+		(property "Sheetname" "Arithmetic Logic Unit"
+			(at 85.09 50.0884 0)
+			(effects
+				(font
+					(size 1.27 1.27)
+				)
+				(justify left bottom)
+			)
+		)
+		(property "Sheetfile" "alu.kicad_sch"
+			(at 85.09 81.8646 0)
+			(effects
+				(font
+					(size 1.27 1.27)
+				)
+				(justify left top)
+			)
+		)
+		(instances
+			(project "CPU_block_diagram"
+				(path "/5324683e-15fd-4fa9-8f28-7726564ef1dc"
+					(page "7")
+				)
+			)
+		)
 	)
 	(sheet

Commit message: vault backup: 2026-01-16 03:08:08
Other:
- sheet Arithmetic Logic Unit ports: added A0, A1, A2, A3, A4, A5, A6, A7, B0, B1, B2, B3, B4, B5, B6, B7; removed none
Changed lines of the file:
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@@
 	)
 	(sheet
-		(at 85.09 50.8)
-		(size 29.21 30.48)
+		(at 85.09 26.67)
+		(size 29.21 54.61)
 		(exclude_from_sim no)
 		(in_bom yes)
@@
 		)
 		(property "Sheetname" "Arithmetic Logic Unit"
-			(at 85.09 50.0884 0)
+			(at 85.09 25.9584 0)
 			(effects
 				(font
@@
 			)
 		)
+		(pin "A0" input
+			(at 85.09 35.56 180)
+			(effects
+				(font
+					(size 1.27 1.27)
+				)
+				(justify left)
+			)
+		)
+		(pin "A1" input
+			(at 85.09 38.1 180)
+			(effects
+				(font
+					(size 1.27 1.27)
+				)
+				(justify left)
+			)
+		)
+		(pin "A2" input
+			(at 85.09 40.64 180)
+			(effects
+				(font
+					(size 1.27 1.27)
+				)
+				(justify left)
+			)
+		)
+		(pin "A3" input
+			(at 85.09 43.18 180)
+			(effects
+				(font
+					(size 1.27 1.27)
+				)
+				(justify left)
+			)
+		)
+		(pin "A4" input
+			(at 85.09 45.72 180)
+			(effects
+				(font
+					(size 1.27 1.27)
+				)
+				(justify left)
+			)
+		)
+		(pin "A5" input
+			(at 85.09 48.26 180)
+			(effects
+				(font
+					(size 1.27 1.27)
+				)
+				(justify left)
+			)
+		)
+		(pin "A6" input
+			(at 85.09 50.8 180)
+			(effects
+				(font
+					(size 1.27 1.27)
+				)
+				(justify left)
+			)
+		)
+		(pin "A7" input
+			(at 85.09 53.34 180)
+			(effects
+				(font
+					(size 1.27 1.27)
+				)
+				(justify left)
+			)
+		)
+		(pin "B0" input
+			(at 85.09 57.15 180)
+			(effects
+				(font
+					(size 1.27 1.27)
+				)
+				(justify left)
+			)
+		)
+		(pin "B1" input
+			(at 85.09 59.69 180)
+			(effects
+				(font
+					(size 1.27 1.27)
+				)
+				(justify left)
+			)
+		)
+		(pin "B2" input
+			(at 85.09 62.23 180)
+			(effects
+				(font
+					(size 1.27 1.27)
+				)
+				(justify left)
+			)
+		)
+		(pin "B3" input
+			(at 85.09 64.77 180)
+			(effects
+				(font
+					(size 1.27 1.27)
+				)
+				(justify left)
+			)
+		)
+		(pin "B4" input
+			(at 85.09 67.31 180)
+			(effects
+				(font
+					(size 1.27 1.27)
+				)
+				(justify left)
+			)
+		)
+		(pin "B5" input
+			(at 85.09 69.85 180)
+			(effects
+				(font
+					(size 1.27 1.27)
+				)
+				(justify left)
+			)
+		)
+		(pin "B6" input
+			(at 85.09 72.39 180)
+			(effects
+				(font
+					(size 1.27 1.27)
+				)
+				(justify left)
+			)
+		)
+		(pin "B7" input
+			(at 85.09 74.93 180)
+			(effects
+				(font
+					(size 1.27 1.27)
+				)
+				(justify left)
+			)
+		)

Commit message: vault backup: 2026-01-16 05:38:33
Parts:
- removed D26, D27, D28, D29, D30, D31, D32, D33: RED, symbol Device:LED
- removed R32, R33, R34, R35, R36, R37, R38, R39: 220, symbol Device:R_US
- added D44, D45, D46, D47, D48, D49, D50, D51: RED, symbol Device:LED
- added R58, R59, R60, R61, R62, R63, R64, R65: 220, symbol Device:R_US
Connections:
- new net: D50.1 (K), R64.1
- new net: D46.1 (K), R60.1
- new net: R58.2, R59.2, R60.2, R61.2, R62.2, R63.2, R64.2, R65.2
- new net: D44.1 (K), R58.1
- new net: D45.1 (K), R59.1
- new net: D48.1 (K), R62.1
- new net: D49.1 (K), R63.1
- new net: D47.1 (K), R61.1
- new net: D51.1 (K), R65.1
Other:
- sheet Arithmetic Logic Unit ports: added BUS0, BUS1, BUS2, BUS3, BUS4, BUS5, BUS6, BUS7, CF, CLK, CLR, SU, ZF, ~{EO}, ~{FI}; removed none
- moved on the sheet: R40, R41, R42, R43, R44, R45, R46, R47
