File: KiCad/CPU_block_diagram/a_register.kicad_sch (KiCad schematic)
At the start: 19 parts, among them U7 74LS245, U8 74LS173, U9 74LS173

Commit message: vault backup: 2026-01-03 00:49:48
Connections:
- net CLK: now also U8.7 (Cp), U9.7 (Cp)
- net CLR: now reaches U9.15 (Mr)
- net CLR: now also U8.15 (Mr)
- net +5V: now reaches U9.16 (VCC)
- net +5V: now also U7.1 (A->B), U7.20 (VCC), U8.16 (VCC)
- net at U9.3 (Q0): now also U7.6 (A4)
- net at U9.4 (Q1): now also U7.7 (A5)
- net at U9.5 (Q2): now also U7.8 (A6)
- net at U9.6 (Q3): now also U7.9 (A7)
- net GND: now reaches U9.8 (GND)
- net GND: now also U7.10 (GND), U8.8 (GND)
- net at U8.3 (Q0): now also U7.2 (A0)
- net at U8.4 (Q1): now also U7.3 (A1)
- net at U8.5 (Q2): now also U7.4 (A2)
- net at U8.6 (Q3): now also U7.5 (A3)
- net ~{AI}: now reaches U7.19 (CE)
Other:
- moved on the sheet: U7, U8, U9

Commit message: vault backup: 2026-01-03 05:08:47
Parts:
- D2, D3, D4, D5, D6, D7, D8, D9: value LED -> RED
- R10, R11, R12, R13, R14, R15, R8, R9: value R_US -> 220
Connections:
- net GND: now also R10.2, R11.2, R12.2, R13.2, R14.2, R15.2, R8.2, R9.2, U8.1 (Oe1), U8.2 (Oe2), U9.1 (Oe1), U9.2 (Oe2)
- net ~{AI}: now also U8.10 (E2), U8.9 (E1), U9.10 (E2), U9.9 (E1); no longer U7.19 (CE)
- net ~{AO}: now also U7.19 (CE)
- net at R8.1: now also D2.1 (K)
- net at R11.1: now also D5.1 (K)
- net A4: now reaches D5.2 (A)
- net A4: now also U7.5 (A3), U8.6 (Q3)
- net A3: now reaches U7.6 (A4), U9.3 (Q0)
- net A3: now also D6.2 (A)
- net A2: now reaches U7.7 (A5), U9.4 (Q1)
- net A2: now also D7.2 (A)
- net A1: now reaches U7.8 (A6), U9.5 (Q2)
- net A1: now also D8.2 (A)
- net A0: now reaches U7.9 (A7), U9.6 (Q3)
- net A0: now also D9.2 (A)
- net A7: now reaches U7.2 (A0), U8.3 (Q0)
- net A7: now also D2.2 (A)
- net A6: now reaches U7.3 (A1), U8.4 (Q1)
- net A6: now also D3.2 (A)
- net A5: now reaches U7.4 (A2), U8.5 (Q2)
- net A5: now also D4.2 (A)
- net at D6.1 (K): now also R12.1
- net at R14.1: now also D8.1 (K)
- net at D9.1 (K): now also R15.1
- net at D7.1 (K): now also R13.1
- net at D3.1 (K): now also R9.1
- net at R10.1: now also D4.1 (K)
Other:
- moved on the sheet: D2, D3, D4, D5, D6, D7, D8, D9, R10, R11, R12, R13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

Commit message: vault backup: 2026-01-03 05:38:52
Connections:
- net A0 renamed B0
- net A1 renamed B1
- net A2 renamed B2
- net A3 renamed B3
- net A4 renamed B4
- net A5 renamed B5
- net A6 renamed B6
- net A7 renamed B7
- net ~{AI} renamed ~{BI}
- net ~{AO} renamed ~{BO}
Other:
- title: (none) -> Register_B
- moved on the sheet: D2, D3, D4, D5, D6, D7, D8, D9, R10, R11, R12, R13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

Commit message: vault backup: 2026-01-03 11:53:08
Parts:
- renumbered D2 to D10, D3 to D11, D4 to D12, D5 to D13, D6 to D14, D7 to D15, D8 to D16, D9 to D17, R8 to R16, U7 to U10, U8 to U11, U9 to U12
Connections:
- net B0 renamed A0
- net B1 renamed A1
- net B2 renamed A2
- net B3 renamed A3
- net B4 renamed A4
- net B5 renamed A5
- net B6 renamed A6
- net B7 renamed A7
- net ~{BI} renamed ~{AI}
- net ~{BO} renamed ~{AO}
Other:
- title: Register_B -> Register_A
Changed lines of the file:
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@@
 	(paper "A4")
 	(title_block
-		(title "Register_B")
+		(title "Register_A")
 	)
 	(text_box "Oe1 and Oe2 will enable the outputs when set to low.\n\nData receives from the bus and latches at Clock Pulse.\n\nQ3 is the least significant bit."
@@
 		)
 	)
-	(hierarchical_label "B6"
+	(hierarchical_label "A6"
 		(shape output)
 		(at 262.89 34.29 0)
@@
 		)
 	)
-	(hierarchical_label "~{BO}"
+	(hierarchical_label "~{AO}"
 		(shape input)
 		(at 36.83 46.99 180)
@@
 		)
 	)
-	(hierarchical_label "B4"
+	(hierarchical_label "A4"
 		(shape output)
 		(at 262.89 29.21 0)
@@
 		)
 	)
-	(hierarchical_label "B1"
+	(hierarchical_label "A1"
 		(shape output)
 		(at 262.89 21.59 0)
@@
 		)
 	)
-	(hierarchical_label "B3"
+	(hierarchical_label "A3"
 		(shape output)
 		(at 262.89 26.67 0)
@@
 		)
 	)
-	(hierarchical_label "B7"
+	(hierarchical_label "A7"
 		(shape output)
 		(at 262.89 36.83 0)
@@
 		)
 	)
-	(hierarchical_label "B0"
+	(hierarchical_label "A0"
 		(shape output)
 		(at 262.89 19.05 0)
@@
 		)
 	)
-	(hierarchical_label "B2"
+	(hierarchical_label "A0"
+		(shape output)
+		(at 262.89 19.05 0)
+		(effects
+			(font
+				(size 1.27 1.27)
+			)
+			(justify left)
+		)
+	)
+	(hierarchical_label "A2"
 		(shape output)
 		(at 262.89 24.13 0)
@@
 		)
 	)
-	(hierarchical_label "B5"
+	(hierarchical_label "A5"
 		(shape output)
 		(at 262.89 31.75 0)
@@
 		)
 	)
-	(hierarchical_label "~{BI}"
+	(hierarchical_label "~{AI}"
 		(shape input)
 		(at 36.83 44.45 180)
@@
 		(dnp no)
 		(fields_autoplaced yes)
-		(property "Reference" "R8"
+		(property "Reference" "R16"
 			(at 113.03 142.2399 0)
 			(effects
@@
 				)
 				(path "/5324683e-15fd-4fa9-8f28-7726564ef1dc/d4c15e47-95e9-40ff-9967-f62269b25945"
-					(reference "R8")
+					(reference "R16")
 					(unit 1)
 				)
@@
 		(dnp no)
 		(fields_autoplaced yes)
-		(property "Reference" "#PWR017"
+		(property "Reference" "#PWR021"
 			(at 107.95 78.74 0)
 			(effects
@@
 			(project "CPU_block_diagram"
 				(path "/5324683e-15fd-4fa9-8f28-7726564ef1dc/a71ef12c-ad37-4d04-9035-f9e49f453cc9"
-					(reference "#PWR023")
+					(reference "#PWR0105")
 					(unit 1)
 				)
 				(path "/5324683e-15fd-4fa9-8f28-7726564ef1dc/d4c15e47-95e9-40ff-9967-f62269b25945"
-					(reference "#PWR017")
+					(reference "#PWR021")
 					(unit 1)
 				)
@@
 		(dnp no)
 		(fields_autoplaced yes)
-		(property "Reference" "D5"
+		(property "Reference" "D13"
 			(at 144.78 132.3974 90)
 			(effects
@@
 				)
 				(path "/5324683e-15fd-4fa9-8f28-7726564ef1dc/d4c15e47-95e9-40ff-9967-f62269b25945"
-					(reference "D5")
+					(reference "D13")
 					(unit 1)
 				)
@@
 		(dnp no)
 		(fields_autoplaced yes)
-		(property "Reference" "U9"
+		(property "Reference" "U12"
 			(at 218.44 62.1598 90)
 			(effects
@@
 				)
 				(path "/5324683e-15fd-4fa9-8f28-7726564ef1dc/d4c15e47-95e9-40ff-9967-f62269b25945"
-					(reference "U9")
+					(reference "U12")
 					(unit 1)
 				)
@@
 		(dnp no)
 		(fields_autoplaced yes)
-		(property "Reference" "U8"
+		(property "Reference" "U11"
 			(at 160.02 62.1598 90)
 			(effects
@@
 				)
 				(path "/5324683e-15fd-4fa9-8f28-7726564ef1dc/d4c15e47-95e9-40ff-9967-f62269b25945"
-					(reference "U8")
+					(reference "U11")
 					(unit 1)
 				)
@@
 		(dnp no)
 		(fields_autoplaced yes)
-		(property "Reference" "D6"
+		(property "Reference" "D14"
 			(at 154.94 132.3974 90)
 			(effects
@@
 				)
 				(path "/5324683e-15fd-4fa9-8f28-7726564ef1dc/d4c15e47-95e9-40ff-9967-f62269b25945"
-					(reference "D6")
+					(reference "D14")
 					(unit 1)
 				)
@@
 		(dnp no)
 		(fields_autoplaced yes)
-		(property "Reference" "D9"
+		(property "Reference" "D17"
 			(at 185.42 132.3974 90)
 			(effects
@@
 				)
 				(path "/5324683e-15fd-4fa9-8f28-7726564ef1dc/d4c15e47-95e9-40ff-9967-f62269b25945"
-					(reference "D9")
+					(reference "D17")
 					(unit 1)
 				)
@@
 		(dnp no)
 		(fields_autoplaced yes)
-		(property "Reference" "#PWR018"
+		(property "Reference" "#PWR022"
 			(at 146.05 158.75 0)
 			(effects
@@
 			(project "CPU_block_diagram"
 				(path "/5324683e-15fd-4fa9-8f28-7726564ef1dc/a71ef12c-ad37-4d04-9035-f9e49f453cc9"
-					(reference "#PWR024")
+					(reference "#PWR0103")
 					(unit 1)
 				)
 				(path "/5324683e-15fd-4fa9-8f28-7726564ef1dc/d4c15e47-95e9-40ff-9967-f62269b25945"
-					(reference "#PWR018")
+					(reference "#PWR022")
 					(unit 1)
 				)
@@
 		(dnp no)
 		(fields_autoplaced yes)
-		(property "Reference" "D7"
+		(property "Reference" "D15"
 			(at 165.1 132.3974 90)
 			(effects
@@
 				)
 				(path "/5324683e-15fd-4fa9-8f28-7726564ef1dc/d4c15e47-95e9-40ff-9967-f62269b25945"
-					(reference "D7")
+					(reference "D15")
 					(unit 1)
 				)
@@
 		(dnp no)
 		(fields_autoplaced yes)
-		(property "Reference" "D3"
+		(property "Reference" "D11"
 			(at 124.46 132.3974 90)
 			(effects
@@
 				)
 				(path "/5324683e-15fd-4fa9-8f28-7726564ef1dc/d4c15e47-95e9-40ff-9967-f62269b25945"
-					(reference "D3")
+					(reference "D11")
 					(unit 1)
 				)
@@
 		(dnp no)
 		(fields_autoplaced yes)
-		(property "Reference" "#PWR016"
+		(property "Reference" "#PWR020"
 			(at 59.69 68.58 0)
 			(effects
@@
 			(project "CPU_block_diagram"
 				(path "/5324683e-15fd-4fa9-8f28-7726564ef1dc/a71ef12c-ad37-4d04-9035-f9e49f453cc9"
-					(reference "#PWR022")
+					(reference "#PWR0106")
 					(unit 1)
 				)
 				(path "/5324683e-15fd-4fa9-8f28-7726564ef1dc/d4c15e47-95e9-40ff-9967-f62269b25945"
-					(reference "#PWR016")
+					(reference "#PWR020")
 					(unit 1)
 				)
@@
 		(dnp no)
 		(fields_autoplaced yes)
-		(property "Reference" "D4"
+		(property "Reference" "D12"
 			(at 134.62 132.3974 90)
 			(effects
@@
 				)
 				(path "/5324683e-15fd-4fa9-8f28-7726564ef1dc/d4c15e47-95e9-40ff-9967-f62269b25945"
-					(reference "D4")
+					(reference "D12")
 					(unit 1)
 				)
@@
 		(dnp no)
 		(fields_autoplaced yes)
-		(property "Reference" "U7"
+		(property "Reference" "U10"
 			(at 101.6 63.1346 90)
 			(effects
@@
 				)
 				(path "/5324683e-15fd-4fa9-8f28-7726564ef1dc/d4c15e47-95e9-40ff-9967-f62269b25945"
-					(reference "U7")
+					(reference "U10")
 					(unit 1)
 				)
@@
 		(dnp no)
 		(fields_autoplaced yes)
-		(property "Reference" "D8"
+		(property "Reference" "D16"
 			(at 175.26 132.3974 90)
 			(effects
@@
 				)
 				(path "/5324683e-15fd-4fa9-8f28-7726564ef1dc/d4c15e47-95e9-40ff-9967-f62269b25945"
-					(reference "D8")
+					(reference "D16")
 					(unit 1)
 				)
@@
 		(dnp no)
 		(fields_autoplaced yes)
-		(property "Reference" "#PWR021"
+		(property "Reference" "#PWR025"
 			(at 226.06 68.58 0)
 			(effects
@@
 			(project "CPU_block_diagram"
 				(path "/5324683e-15fd-4fa9-8f28-7726564ef1dc/a71ef12c-ad37-4d04-9035-f9e49f453cc9"
-					(reference "#PWR027")
+					(reference "#PWR0104")
 					(unit 1)
 				)
 				(path "/5324683e-15fd-4fa9-8f28-7726564ef1dc/d4c15e47-95e9-40ff-9967-f62269b25945"
-					(reference "#PWR021")
+					(reference "#PWR025")
 					(unit 1)
 				)
@@
 		(dnp no)
 		(fields_autoplaced yes)
-		(property "Reference" "#PWR020"
+		(property "Reference" "#PWR024"
 			(at 172.72 78.74 0)
 			(effects
@@
 			(project "CPU_block_diagram"
 				(path "/5324683e-15fd-4fa9-8f28-7726564ef1dc/a71ef12c-ad37-4d04-9035-f9e49f453cc9"
-					(reference "#PWR026")
+					(reference "#PWR0102")
 					(unit 1)
 				)
 				(path "/5324683e-15fd-4fa9-8f28-7726564ef1dc/d4c15e47-95e9-40ff-9967-f62269b25945"
-					(reference "#PWR020")
+					(reference "#PWR024")
 					(unit 1)
 				)
@@
 		(dnp no)
 		(fields_autoplaced yes)
-		(property "Reference" "D2"
+		(property "Reference" "D10"
 			(at 114.3 132.3974 90)
 			(effects
@@
 				)
 				(path "/5324683e-15fd-4fa9-8f28-7726564ef1dc/d4c15e47-95e9-40ff-9967-f62269b25945"
-					(reference "D2")
+					(reference "D10")
 					(unit 1)
 				)
@@
 		(dnp no)
 		(fields_autoplaced yes)
-		(property "Reference" "#PWR019"
+		(property "Reference" "#PWR023"
 			(at 167.64 68.58 0)
 			(effects
@@
 			(project "CPU_block_diagram"
 				(path "/5324683e-15fd-4fa9-8f28-7726564ef1dc/a71ef12c-ad37-4d04-9035-f9e49f453cc9"
-					(reference "#PWR025")
+					(reference "#PWR0101")
 					(unit 1)
 				)
 				(path "/5324683e-15fd-4fa9-8f28-7726564ef1dc/d4c15e47-95e9-40ff-9967-f62269b25945"
-					(reference "#PWR019")
+					(reference "#PWR023")
 					(unit 1)
 				)
