File: KiCad/CPU_block_diagram/a_register.kicad_sch (KiCad schematic)
At the start: 20 parts, among them U10 74LS245, U11 74LS173, U12 74LS173

Commit message: vault backup: 2026-01-05 18:47:29
Connections:
- net A0: now also U12.3 (Q0); no longer U12.6 (Q3)
- net A1: now also U12.4 (Q1); no longer U12.5 (Q2)
- net A2: now also U12.5 (Q2); no longer U12.4 (Q1)
- net A3: now also U12.6 (Q3); no longer U12.3 (Q0)
- net A4: now also U11.3 (Q0); no longer U11.6 (Q3)
- net A5: now also U11.4 (Q1); no longer U11.5 (Q2)
- net A6: now also U11.5 (Q2); no longer U11.4 (Q1)
- net A7: now also U11.6 (Q3); no longer U11.3 (Q0)

Commit message: vault backup: 2026-01-10 22:03:55
Other:
- title: Register_A -> A_Register
Changed lines of the file:
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@@
 	(paper "A4")
 	(title_block
-		(title "Register_A")
+		(title "A_Register")
 	)
 	(rectangle
