File: KiCad/CPU_block_diagram/IR_register.kicad_sch (KiCad schematic)
At the start: 20 parts, among them U10 74LS245, U11 74LS173, U12 74LS173

Commit message: vault backup: 2026-01-03 13:53:37
Parts:
- removed C7: 0.1µF, symbol Device:C
- removed D10, D11, D12, D13, D14, D15, D16, D17: RED, symbol Device:LED
- removed R10, R11, R12, R13, R14, R15, R16, R9: 220, symbol Device:R_US
- removed U10: 74LS245, symbol 74xx:74LS245
- removed U11, U12: 74LS173, symbol 74xx:74LS173
- added C9: 0.1µF, symbol Device:C
- added D18, D19, D20, D21, D22, D23, D24, D25: RED, symbol Device:LED
- added R24, R25, R26, R27, R28, R29, R30, R31: 220, symbol Device:R_US
- added U13: 74LS245, symbol 74xx:74LS245
- added U14, U15: 74LS173, symbol 74xx:74LS173
Connections:
- net +5V: now also C9.1, U13.1 (A->B), U13.20 (VCC), U14.16 (VCC), U15.16 (VCC)
- net BUS0: now also U13.11 (B7), U15.11 (D3)
- net BUS1: now also U13.12 (B6), U15.12 (D2)
- net BUS2: now also U13.13 (B5), U15.13 (D1)
- net BUS3: now also U13.14 (B4), U15.14 (D0)
- net BUS4: now also U13.15 (B3), U14.11 (D3)
- net BUS5: now also U13.16 (B2), U14.12 (D2)
- net BUS6: now also U13.17 (B1), U14.13 (D1)
- net BUS7: now also U13.18 (B0), U14.14 (D0)
- net CLK: now also U14.7 (Cp), U15.7 (Cp)
- net CLR: now also U14.15 (Mr), U15.15 (Mr)
- net GND: now also C9.2, R24.2, R25.2, R26.2, R27.2, R28.2, R29.2, R30.2, R31.2, U13.10 (GND), U14.1 (Oe1), U14.2 (Oe2), U14.8 (GND), U15.1 (Oe1), U15.2 (Oe2), U15.8 (GND)
- new net: D20.1 (K), R26.1
- new net: D18.1 (K), R24.1
- new net: D25.1 (K), R31.1
- new net: D25.2 (A), U13.9 (A7), U15.6 (Q3)
- new net: D23.1 (K), R29.1
- new net: D23.2 (A), U13.7 (A5), U15.4 (Q1)
- new net: D21.1 (K), R27.1
- new net: D19.1 (K), R25.1
- new net: D22.2 (A), U13.6 (A4), U15.3 (Q0)
- new net: D24.2 (A), U13.8 (A6), U15.5 (Q2)
- new net: D22.1 (K), R28.1
- new net: D24.1 (K), R30.1
- new net IR4: D21.2 (A), U13.5 (A3), U14.6 (Q3)
- new net IR5: D20.2 (A), U13.4 (A2), U14.5 (Q2)
- new net IR6: D19.2 (A), U13.3 (A1), U14.4 (Q1)
- new net IR7: D18.2 (A), U13.2 (A0), U14.3 (Q0)
- new net ~{IRI}: U14.10 (E2), U14.9 (E1), U15.10 (E2), U15.9 (E1)
- new net ~{IRO}: U13.19 (CE)
Other:
- title: Register_A -> (none)

Commit message: vault backup: 2026-01-05 18:47:29
Connections:
- net IR4: now also U14.3 (Q0); no longer U14.6 (Q3)
- net IR5: now also U14.4 (Q1); no longer U14.5 (Q2)
- net IR6: now also U14.5 (Q2); no longer U14.4 (Q1)
- net IR7: now also U14.6 (Q3); no longer U14.3 (Q0)
- new net: D25.2 (A), U15.3 (Q0)
- new net: D23.2 (A), U15.5 (Q2)
- new net: D24.2 (A), U15.4 (Q1)
- new net: D22.2 (A), U15.6 (Q3)
- now unconnected: U13.6 (A4), U13.7 (A5), U13.8 (A6), U13.9 (A7)

Commit message: vault backup: 2026-01-06 02:33:08
Parts:
- D18, D19, D20, D21: value RED -> BLUE
- D22, D23, D24, D25: value RED -> YELLOW
Connections:
- net at D25.2 (A), U15.3 (Q0): now also U13.9 (A7)
- net at D23.2 (A), U15.5 (Q2): now also U13.7 (A5)
- net at D24.2 (A), U15.4 (Q1): now also U13.8 (A6)
- net at D22.2 (A), U15.6 (Q3): now also U13.6 (A4)

Commit message: vault backup: 2026-01-10 22:03:55
Other:
- title: (none) -> Instruction_Register
Changed lines of the file:
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@@
 	(generator_version "9.0")
 	(paper "A4")
+	(title_block
+		(title "Instruction_Register")
+	)
 	(rectangle
 		(start 16.51 144.78)
