File: KiCad/CPU_block_diagram/b_register.kicad_sch (KiCad schematic)
At the start: 0 parts

Commit message: vault backup: 2026-01-03 13:53:37
Parts:
- added C8: 0.1µF, symbol Device:C
- added D2, D3, D4, D5, D6, D7, D8, D9: RED, symbol Device:LED
- added R17, R18, R19, R20, R21, R22, R23, R8: 220, symbol Device:R_US
- added U7: 74LS245, symbol 74xx:74LS245
- added U8, U9: 74LS173, symbol 74xx:74LS173
Connections:
- new net: D8.1 (K), R22.1
- new net: D9.1 (K), R23.1
- new net: D5.1 (K), R19.1
- new net: D2.1 (K), R8.1
- new net: D3.1 (K), R17.1
- new net: D7.1 (K), R21.1
- new net: D6.1 (K), R20.1
- new net: D4.1 (K), R18.1
- new net +5V: C8.1, U7.1 (A->B), U7.20 (VCC), U8.16 (VCC), U9.16 (VCC)
- new net B0: D9.2 (A), U7.9 (A7), U9.6 (Q3)
- new net B1: D8.2 (A), U7.8 (A6), U9.5 (Q2)
- new net B2: D7.2 (A), U7.7 (A5), U9.4 (Q1)
- new net B3: D6.2 (A), U7.6 (A4), U9.3 (Q0)
- new net B4: D5.2 (A), U7.5 (A3), U8.6 (Q3)
- new net B5: D4.2 (A), U7.4 (A2), U8.5 (Q2)
- new net B6: D3.2 (A), U7.3 (A1), U8.4 (Q1)
- new net B7: D2.2 (A), U7.2 (A0), U8.3 (Q0)
- new net BUS0: U7.11 (B7), U9.11 (D3)
- new net BUS1: U7.12 (B6), U9.12 (D2)
- new net BUS2: U7.13 (B5), U9.13 (D1)
- new net BUS3: U7.14 (B4), U9.14 (D0)
- new net BUS4: U7.15 (B3), U8.11 (D3)
- new net BUS5: U7.16 (B2), U8.12 (D2)
- new net BUS6: U7.17 (B1), U8.13 (D1)
- new net BUS7: U7.18 (B0), U8.14 (D0)
- new net CLK: U8.7 (Cp), U9.7 (Cp)
- new net CLR: U8.15 (Mr), U9.15 (Mr)
- new net GND: C8.2, R17.2, R18.2, R19.2, R20.2, R21.2, R22.2, R23.2, R8.2, U7.10 (GND), U8.1 (Oe1), U8.2 (Oe2), U8.8 (GND), U9.1 (Oe1), U9.2 (Oe2), U9.8 (GND)
- new net ~{BI}: U8.10 (E2), U8.9 (E1), U9.10 (E2), U9.9 (E1)
- new net ~{BO}: U7.19 (CE)
Other:
- note added: "Decoupler"

Commit message: vault backup: 2026-01-05 18:47:29
Connections:
- net B0: now also U9.3 (Q0); no longer U9.6 (Q3)
- net B1: now also U9.4 (Q1); no longer U9.5 (Q2)
- net B2: now also U9.5 (Q2); no longer U9.4 (Q1)
- net B3: now also U9.6 (Q3); no longer U9.3 (Q0)
- net B4: now also U8.3 (Q0); no longer U8.6 (Q3)
- net B5: now also U8.4 (Q1); no longer U8.5 (Q2)
- net B6: now also U8.5 (Q2); no longer U8.4 (Q1)
- net B7: now also U8.6 (Q3); no longer U8.3 (Q0)

Commit message: vault backup: 2026-01-10 22:03:55
Other:
- title: (none) -> B_Register
Changed lines of the file:
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@@
 	(generator_version "9.0")
 	(paper "A4")
+	(title_block
+		(title "B_Register")
+	)
 	(rectangle
 		(start 16.51 144.78)
