File: KiCad/CPU_block_diagram/_autosave-alu.kicad_sch (KiCad schematic)
At the start: 8 parts, among them U16 74LS245, U17 74LS283, U18 74LS283, U19 74LS86, U20 74LS86, U21 74LS02, U22 74LS08

Commit message: vault backup: 2026-01-15 03:11:46
Connections:
- net at U20.5: now also U18.7 (C0), U19.10, U19.13, U19.2, U19.5, U20.10, U20.13, U20.2
- net at U20.6: now also U18.14 (A3); no longer U18.2 (B2)
- net at U18.11 (B4): no longer U20.11
- net at U18.15 (B3): no longer U20.8
- net at U18.3 (A2): now also U20.8
- net at U18.5 (A1): now also U20.11
Other:
- moved on the sheet: U17, U18, U19A, U19B, U19C, U19D, U20A, U20B, U20C, U20D

Commit message: vault backup: 2026-01-15 03:26:50
Connections:
- net at U20.6: now also U18.15 (B3); no longer U18.14 (A3)
- net at U19.11: now also U17.6 (B1)
- net at U17.11 (B4): now also U19.3
- net at U17.15 (B3): now also U19.6
- net at U17.2 (B2): now also U19.8
- net at U18.11 (B4): now also U20.3
- net at U18.2 (B2): now also U20.8
- net at U18.3 (A2): no longer U20.8
- net at U18.5 (A1): no longer U20.11
- net at U18.6 (B1): now also U20.11
Other:
- moved on the sheet: U19A, U19B, U19C, U20A, U20B, U20C, U20D

Commit message: vault backup: 2026-01-15 03:41:55
Connections:
- net at U20.6: no longer U18.15 (B3)
- net at U19.11: no longer U17.6 (B1)
- net at U17.11 (B4): no longer U19.3
- net at U17.15 (B3): no longer U19.6
- net at U17.2 (B2): no longer U19.8
- net at U17.7 (C0): no longer U18.9 (C4)
- net at U18.11 (B4): no longer U20.3
- net at U18.2 (B2): no longer U20.8
- net at U18.6 (B1): no longer U20.11
Other:
- moved on the sheet: U17, U18
