File: KiCad/CPU_block_diagram/_autosave-alu.kicad_sch (KiCad schematic)
At the start: 8 parts, among them U16 74LS245, U17 74LS283, U18 74LS283, U19 74LS86, U20 74LS86, U21 74LS02, U22 74LS08

Commit message: vault backup: 2026-01-15 18:57:41
Parts:
- added D34, D35, D36, D37, D38, D39, D40, D41: RED, symbol Device:LED
- added R48, R49, R50, R51, R52, R53, R54, R55: 220, symbol Device:R_US
- added U23: 74LS173, symbol 74xx:74LS173
Connections:
- net GND: now also U16.10 (GND), R48.2, R49.2, R50.2, R51.2, R52.2, R53.2, R54.2, R55.2
- net VCC: now also U16.1 (A->B), U16.20 (VCC)
- net SU: now reaches U19.10, U19.13, U19.2, U19.5, U20.10, U20.13, U20.2, U20.5
- net at U21.11: now also U16.9 (A7)
- net at U21.12: now also U16.8 (A6)
- net BUS0: now reaches U16.11 (B7)
- net BUS1: now reaches U16.12 (B6)
- net BUS2: now reaches U16.13 (B5)
- net BUS3: now reaches U16.14 (B4)
- net BUS4: now reaches U16.15 (B3)
- net BUS5: now reaches U16.16 (B2)
- net BUS6: now reaches U16.17 (B1)
- net BUS7: now reaches U16.18 (B0)
- net ~{EO}: now reaches U16.19 (CE)
- net at U16.2 (A0): now also U21.3
- net at U16.3 (A1): now also U21.2
- net at U16.4 (A2): now also U21.6
- net at U16.5 (A3): now also U21.5
- net at U16.6 (A4): now also U21.9
- net at U16.7 (A5): now also U21.8
- new net: D38.1 (K), R52.1
- new net: D40.1 (K), R54.1
- new net: D41.1 (K), R55.1
- new net: D39.1 (K), R53.1
- new net: D36.1 (K), R50.1
- new net: D35.1 (K), R49.1
- new net: D37.1 (K), R51.1
- new net: D34.1 (K), R48.1
Other:
- moved on the sheet: U16, U21A, U21B, U21C, U21D, U22A, U22B, U22C
